File: MainModule.brd (EAGLE design)
At the start: 87.6 x 49.5 mm, 75 parts, among them IC1 LPC1764, IC2 KSZ8001L, IC4 REG1117, IC5 7805, IC6 74LVC1G04, J1 USBSMD, J2 POWER_JACKPTH, J3 MAGJACK-SI-52008, Q1 BSS84, Q2 MOSFET-NCHANNELSMD, U1 HVPS-1363, U2 7W-50.000MBB-T, Y1 32.768KHz, Y2 12MHz

Commit message: manufacture-ready
Parts:
- Q2: value MOSFET-NCHANNELSMD -> 2N7002
- moved JP9 0.57 mm to (61.0, 16.3)
- moved R16 0.25 mm to (56.1, 25.7)
- moved R20 0.13 mm to (39.0, 32.0)
Connections:
- net JP7_5: now also IC1.52; no longer IC1.51
- net JP7_8: now also IC1.51; no longer IC1.52
Routing:
- net GND: track 4.84 -> 24.7 mm
- net N$29: track 22.8 -> 9.79 mm, vias 0 -> 1
- net JP7_8: track 19.1 -> 16.0 mm
- net ENET_TX_EN: track 16.2 -> 14.3 mm
- net ENET_REF_CLK: track 21.9 -> 23.8 mm
- net ENET_RX_ER: track 16.6 -> 18.1 mm
- net RSTOUT: track 35.9 -> 37.3 mm
- net +3V3: track 262.5 -> 263.7 mm
- net 5V: track 122.1 -> 123.2 mm
- net ENET_MDC: track 16.2 -> 17.3 mm
- net OUT_ENA: track 34.0 -> 35.0 mm
- net ENET_MDIO: track 25.2 -> 26.0 mm
- net JP7_7: track 39.4 -> 38.6 mm
- net JP7_6: track 17.3 -> 16.5 mm
- net USB_VBUS: track 55.5 -> 56.1 mm
Other:
- board text added: "P0[0]"
- board text added: "P0[10]"
- board text added: "P0[11]"
- board text added: "P0[15]"
- board text added: "P0[16]"
- board text added: "P0[17]"
- board text added: "P0[18]"
- board text added: "P0[19]"
- board text added: "P0[1]"
- board text added: "P0[20]"
- board text added: "P0[21]"
- board text added: "P0[22]"
- board text added: "P1[19]"
- board text added: "P1[20]"
- board text added: "P1[21]"
- board text added: "P1[22]"
- board text added: "P1[23]"
- board text added: "P1[24]"
- board text added: "P1[25]"
- board text added: "P1[26]"
- board text added: "P2[10]"
- board text added: "P2[11]"
- board text added: "P2[12]"
- board text added: "P2[13]"
- board text added: "RX"
- board text added: "TX"
- board text added: "http://git.io/kpS-Pw"

Commit message: Rev B
Parts:
- removed C24: 10uF, rcl:PANASONIC_B
- removed IC5: 7805, linear:TO220V
- removed IC6: 74LVC1G04, mylib:SOT-25
- removed Q2: 2N7002, SparkFun:SOT23-3
- removed U2: 7W-50.000MBB-T, SparkFun:CRYSTAL-SMD-7X5
- added C13: 100nF, SparkFun:0805
- added C25, C26: 12pF, SparkFun:0805
- added D2: (no value), diode:SMB
- added IC3: KSZ8051RNL, mylib:QFN-32
- added L1: (no value), mylib:INDUCTOR-MCSDC0906
- added PWR, USB: (no value), led:CHIP-LED0805
- added R22: 100k, SparkFun:0805
- added R27, R28: 330, SparkFun:0805
- added Y3: 25MHz, mylib:TXC-7A
- C10: value 1uF -> (none); device SparkFun:0805 -> SparkFun:PANASONIC_D
- C18: value 100nF -> 18p
- C2, C3: value 12pF -> 5p
- C21: value 10uF -> 18p
- C8, C9: value 1uF -> 100nF
- IC2: value KSZ8001L -> MIC4680; device mylib:LQFP48-7X7 -> BillPorter:SOIC-8
- R13: value 4.7k -> 10k
- R15: value 10k -> (none)
- R16: value 2.2k -> (none)
- R20: value 10k -> 47k
- R21: value (none) -> 330
- R6: value 6.65k -> 6.49k
- Y1: device crystal:TC26V -> mylib:85SMX
- moved R15 39.2 mm to (18.5, 25.7), turned to 0 degrees
- moved IC2 34.3 mm to (22.6, 21.6)
- moved C21 34.1 mm to (71.6, 19.6), turned to 180 degrees
- moved R16 33.8 mm to (22.4, 25.7), turned to 180 degrees
- moved R17 24.4 mm to (5.33, 27.4), turned to 270 degrees
- moved C17 24.0 mm to (62.2, 21.1), turned to 0 degrees
- moved C10 22.8 mm to (29.0, 36.8), turned to 180 degrees
- moved R14 21.4 mm to (57.1, 22.6), turned to 180 degrees
- moved C18 19.3 mm to (71.6, 17.0), turned to 180 degrees
- moved C8 19.3 mm to (62.2, 25.7)
- moved R18 16.1 mm to (57.9, 44.2), turned to 90 degrees
- moved IC4 15.1 mm to (32.8, 44.2), turned to 270 degrees
- moved R11 14.7 mm to (75.2, 22.4), turned to 180 degrees
- moved R12 13.2 mm to (71.6, 22.4), turned to 180 degrees
- moved C12 12.6 mm to (65.0, 24.9), turned to 90 degrees
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Connections:
- net N$4 renamed HV
- removed net N$39: Q2.3, R21.1
- new net BTN1: IC1.45
- new net ENET_RST: C17.1, IC1.77, IC3.32, R14.1
- new net LED1: IC1.27, R21.2
- new net N$4: R27.1, USB.A
- new net N$43: D2.C, IC2.3, L1.1
- new net N$44: IC1.18, R22.1
- new net N$7: PWR.A, R28.1
- new net USB_LED: IC1.32, R27.2
- net +3V3: now also IC3.17, IC3.3, R13.2, R14.2, R28.2; no longer C17.1, C18.1, IC2.24, IC2.38, IC2.7, IC6.5, LED1.A, R13.1, R14.1, R15.1, R16.1, U2.P$1, U2.P$4
- net 5V: now also C10.+, L1.4, R15.1; no longer C24.+, IC5.3
- net ENET_CRS: now also IC3.18; no longer IC2.9
- net ENET_LED_0: now also IC3.30; no longer IC2.26
- net ENET_LED_1: now also IC3.31; no longer IC2.27
- net ENET_MDC: now also IC3.12; no longer IC2.2
- net ENET_MDIO: now also IC3.11; no longer IC2.1, R16.2
- net ENET_RD_N: now also IC3.4; no longer IC2.32
- net ENET_RD_P: now also IC3.5; no longer IC2.33
- net ENET_REF_CLK: now also IC3.19; no longer IC2.15, IC6.4
- net ENET_RXD0: now also IC3.16; no longer IC2.6
- net ENET_RXD1: now also IC3.15; no longer IC2.5
- net ENET_RX_ER: now also IC3.20; no longer IC2.11
- net ENET_TD_N: now also IC3.6; no longer IC2.40
- net ENET_TD_P: now also IC3.7; no longer IC2.41
- net ENET_TXD0: now also IC3.24; no longer IC2.17
- net ENET_TXD1: now also IC3.25; no longer IC2.18
- net ENET_TX_EN: now also IC3.23; no longer IC2.16
- net GND: now also C10.-, C13.2, C25.2, C26.2, C8.2, C9.2, D2.A, IC2.1, IC2.5, IC2.6, IC2.7, IC3.1, IC3.22, IC3.26, IC3.27, IC3.EP, LED1.C, PWR.C, R16.1, USB.C; no longer C10.1, C24.-, C8.1, C9.1, IC2.12, IC2.23, IC2.35, IC2.36, IC2.39, IC2.44, IC5.2, IC6.3, Q2.2, U2.P$2
- net JP6_8: now also IC1.48; no longer IC1.47
- net JP6_9: now also IC1.47; no longer IC1.48
- net N$2: now also IC2.2; no longer IC5.1
- net N$23: now also Y1.1; no longer Y1.2
- net N$24: now also R22.2, Y1.4; no longer IC1.18, Y1.1
- net N$25: now also IC3.10, R6.2; no longer C10.2, C8.2, C9.2, IC2.13, IC2.31, IC2.47
- net N$28: now also C25.1, IC3.9, Y3.P$2; no longer IC2.37, R6.2
- net N$30: now also C26.1, IC3.8, Y3.P$1; no longer IC2.21, R13.2
- net N$32: now also C8.1, C9.1, IC3.2; no longer IC6.2, U2.P$3
- net N$37: now also IC3.28, R13.1; no longer IC2.46, R15.2
- net N$38: now also LED1.A, R21.1; no longer LED1.C, R21.2
- net N$42: now also IC2.4, R15.2, R16.2; no longer IC1.24, Q2.1
- net RESET: now also C13.1
- net RSTOUT: now also IC1.6; no longer C21.1, IC1.14, IC2.48, R14.2
- net SWDCLK: now also IC1.5
- net USB_D_N: now also C18.1
- net USB_D_P: now also C21.1
Routing:
- net GND: track 24.7 -> 84.5 mm, vias 34 -> 50
- net 5V: track 123.2 -> 168.3 mm
- net RSTOUT: track 37.3 -> 0.00 mm
- net ENET_LED_0: track 5.94 -> 31.0 mm
- net ENET_LED_1: track 8.06 -> 32.8 mm
- net N$25: track 30.6 -> 11.0 mm
- net SWDCLK: track 0.00 -> 19.2 mm
- net ENET_RST: track 0.00 -> 17.9 mm, vias 0 -> 2
- net OUT_ENA: track 35.0 -> 50.2 mm, vias 0 -> 1
- net N$29: track 9.79 -> 23.8 mm, vias 1 -> 0
- net RESET: track 23.5 -> 37.5 mm
- net ENET_REF_CLK: track 23.8 -> 10.5 mm, vias 2 -> 0
- net ENET_TD_N: track 33.1 -> 19.9 mm
- net N$43: track 0.00 -> 10.8 mm
- net ENET_TXD0: track 8.82 -> 18.7 mm, vias 0 -> 2
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Other:
- board text added: "P0"
- board text added: "P1"
- board text added: "P2"
- board text added: "REV C"
- board text added: "[0]"
- board text added: "[10]"
- board text added: "[11]"
- board text added: "[12]"
- board text added: "[13]"
- board text added: "[15]"
- board text added: "[16]"
- board text added: "[17]"
- board text added: "[18]"
- board text added: "[19]"
- board text added: "[1]"
- board text added: "[20]"
- board text added: "[21]"
- board text added: "[22]"
- board text added: "[23]"
- board text added: "[24]"
- board text added: "[25]"
- board text added: "[26]"
- board text removed: "P0[0]"
- board text removed: "P0[10]"
- board text removed: "P0[11]"
- board text removed: "P0[15]"
- board text removed: "P0[16]"
- board text removed: "P0[17]"
- board text removed: "P0[18]"
- board text removed: "P0[19]"
- board text removed: "P0[1]"
- board text removed: "P0[20]"
- board text removed: "P0[21]"
- board text removed: "P0[22]"
- board text removed: "P1[19]"
- board text removed: "P1[20]"
- board text removed: "P1[21]"
- board text removed: "P1[22]"
- board text removed: "P1[23]"
- board text removed: "P1[24]"
- board text removed: "P1[25]"
- board text removed: "P1[26]"
- board text removed: "P2[10]"
- board text removed: "P2[11]"
- board text removed: "P2[12]"
- board text removed: "P2[13]"
- board text removed: "REV A"
