File: MainModule.sch (EAGLE design)
At the start: 74 parts, among them IC1 LPC1764, IC2 KSZ8001L, IC4 REG1117, IC5 7805, IC6 74LVC1G04, J1 USBSMD, J2 POWER_JACKPTH, J3 MAGJACK-SI-52008, Q1 BSS84, Q2 MOSFET-NCHANNELSMD, U1 HVPS-1363, U2 7W-50.000MBB-T, Y1 32.768KHz, Y2 12MHz

Commit message: manufacture-ready
Parts:
- Q2: value MOSFET-NCHANNELSMD -> 2N7002
Connections:
- net JP7_5: now also IC1.P2[11]/EINT1/I2STX_CLK; no longer IC1.P2[12]/EINT2/I2STX_WS
- net JP7_8: now also IC1.P2[12]/EINT2/I2STX_WS; no longer IC1.P2[11]/EINT1/I2STX_CLK
Other:
- note added: "JP6-H: P0[0], P0[1], p0[10], P0[11]"
- moved on the sheet: C12
Changed lines of the file:
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@@
 <part name="+3V12" library="supply1" deviceset="+3V3" device=""/>
 <part name="BAT" library="pinhead" deviceset="PINHD-1X2" device=""/>
-<part name="Q2" library="SparkFun" deviceset="MOSFET-NCHANNEL" device="SMD"/>
+<part name="Q2" library="SparkFun" deviceset="MOSFET-NCHANNEL" device="SMD" value="2N7002"/>
 <part name="GND7" library="supply1" deviceset="GND" device=""/>
 </parts>
@@
 <wire x1="355.6" y1="-27.94" x2="355.6" y2="43.18" width="0.1524" layer="97"/>
 <wire x1="307.34" y1="-27.94" x2="193.04" y2="-27.94" width="0.1524" layer="97"/>
+<text x="45.72" y="137.16" size="1.778" layer="91">JP6-H: P0[0], P0[1], p0[10], P0[11]</text>
 </plain>
 <instances>
@@
 <instance part="R12" gate="G$1" x="276.86" y="157.48"/>
 <instance part="+3V4" gate="G$1" x="177.8" y="167.64"/>
-<instance part="C12" gate="G$1" x="177.8" y="157.48" rot="R180"/>
-<instance part="GND15" gate="1" x="177.8" y="147.32"/>
+<instance part="C12" gate="G$1" x="177.8" y="144.78" rot="R180"/>
+<instance part="GND15" gate="1" x="177.8" y="132.08"/>
 <instance part="+3V5" gate="G$1" x="185.42" y="63.5"/>
 <instance part="R13" gate="G$1" x="281.94" y="81.28" rot="R270"/>
@@
 <segment>
 <pinref part="+3V4" gate="G$1" pin="+3V3"/>
-<wire x1="177.8" y1="165.1" x2="177.8" y2="162.56" width="0.1524" layer="91"/>
-<wire x1="177.8" y1="162.56" x2="187.96" y2="162.56" width="0.1524" layer="91"/>
+<wire x1="177.8" y1="165.1" x2="177.8" y2="154.94" width="0.1524" layer="91"/>
+<wire x1="177.8" y1="154.94" x2="190.5" y2="154.94" width="0.1524" layer="91"/>
 <pinref part="C12" gate="G$1" pin="2"/>
-<wire x1="177.8" y1="160.02" x2="177.8" y2="162.56" width="0.1524" layer="91"/>
-<junction x="177.8" y="162.56"/>
-<junction x="177.8" y="162.56"/>
+<wire x1="177.8" y1="147.32" x2="177.8" y2="154.94" width="0.1524" layer="91"/>
+<junction x="177.8" y="154.94"/>
+<junction x="177.8" y="154.94"/>
 <wire x1="220.98" y1="154.94" x2="190.5" y2="154.94" width="0.1524" layer="91"/>
-<wire x1="190.5" y1="154.94" x2="187.96" y2="154.94" width="0.1524" layer="91"/>
-<wire x1="187.96" y1="154.94" x2="187.96" y2="162.56" width="0.1524" layer="91"/>
 <pinref part="J3" gate="G$1" pin="CT"/>
 <pinref part="R9" gate="G$1" pin="1"/>
@@
 <pinref part="GND15" gate="1" pin="GND"/>
 <pinref part="C12" gate="G$1" pin="1"/>
-<wire x1="177.8" y1="149.86" x2="177.8" y2="152.4" width="0.1524" layer="91"/>
+<wire x1="177.8" y1="134.62" x2="177.8" y2="139.7" width="0.1524" layer="91"/>
 </segment>
 <segment>
@@
 <net name="JP7_8" class="0">
 <segment>
-<pinref part="IC1" gate="G$1" pin="P2[11]/EINT1/I2STX_CLK"/>
-<wire x1="142.24" y1="30.48" x2="149.86" y2="30.48" width="0.1524" layer="91"/>
-</segment>
-<segment>
 <pinref part="JP7" gate="A" pin="4"/>
 <wire x1="-81.28" y1="22.86" x2="-76.2" y2="22.86" width="0.1524" layer="91"/>
+</segment>
+<segment>
+<pinref part="IC1" gate="G$1" pin="P2[12]/EINT2/I2STX_WS"/>
+<wire x1="142.24" y1="27.94" x2="149.86" y2="27.94" width="0.1524" layer="91"/>
 </segment>
 </net>
@@
 <net name="JP7_5" class="0">
 <segment>
-<pinref part="IC1" gate="G$1" pin="P2[12]/EINT2/I2STX_WS"/>
-<wire x1="142.24" y1="27.94" x2="149.86" y2="27.94" width="0.1524" layer="91"/>
-</segment>
-<segment>
 <pinref part="JP7" gate="A" pin="1"/>
 <wire x1="-88.9" y1="25.4" x2="-93.98" y2="25.4" width="0.1524" layer="91"/>
 </segment>
+<segment>
+<pinref part="IC1" gate="G$1" pin="P2[11]/EINT1/I2STX_CLK"/>
+<wire x1="142.24" y1="30.48" x2="149.86" y2="30.48" width="0.1524" layer="91"/>
+</segment>
 </net>
 <net name="JP6_9" class="0">
@@
 <segment>
 <pinref part="IC1" gate="G$1" pin="P1[19]/MCOA0/USB_PPWR/CAP1[1]"/>
-<wire x1="142.24" y1="93.98" x2="152.4" y2="93.98" width="0.1524" layer="91"/>
+<wire x1="142.24" y1="93.98" x2="154.94" y2="93.98" width="0.1524" layer="91"/>
 </segment>
 </net>
@@
 <segment>
 <pinref part="IC1" gate="G$1" pin="P1[21]/MCABORT/PWM1[3]/SSEL0"/>
-<wire x1="142.24" y1="88.9" x2="152.4" y2="88.9" width="0.1524" layer="91"/>
+<wire x1="142.24" y1="88.9" x2="154.94" y2="88.9" width="0.1524" layer="91"/>
 </segment>
 </net>
@@
 <segment>
 <pinref part="IC1" gate="G$1" pin="P1[20]/MCI0/PWM1[2]/SCK0"/>
-<wire x1="142.24" y1="91.44" x2="152.4" y2="91.44" width="0.1524" layer="91"/>
+<wire x1="142.24" y1="91.44" x2="154.94" y2="91.44" width="0.1524" layer="91"/>
 </segment>
 </net>
@@
 <segment>
 <pinref part="IC1" gate="G$1" pin="P1[22]/MCOB0/USB_PWRD/MAT1[0]"/>
-<wire x1="142.24" y1="86.36" x2="152.4" y2="86.36" width="0.1524" layer="91"/>
-</segment>
-</net>
+<wire x1="142.24" y1="86.36" x2="154.94" y2="86.36" width="0.1524" layer="91"/>
+</segment>
+</net>

Commit message: Rev B
Parts:
- removed C24: 10uF, rcl:CPOL-EUB
- removed IC5: 7805, linear:7805TV
- removed IC6: 74LVC1G04, mylib:74LVC1G04
- removed Q2: 2N7002, SparkFun:MOSFET-NCHANNELSMD
- removed U2: 7W-50.000MBB-T, SparkFun:OSCILLATORSMD
- added C13: 100nF, SparkFun:CAP0805
- added C25, C26: 12pF, SparkFun:CAP0805
- added D2: (no value), diode:SCHOTTKY-DIODESMD
- added IC3: KSZ8051RNL, mylib:KSZ8051RNL
- added L1: (no value), mylib:INDUCTORB
- added PWR, USB: (no value), led:LEDCHIP-LED0805
- added R22: 100k, SparkFun:RESISTOR0805-RES
- added R27, R28: 330, SparkFun:RESISTOR0805-RES
- added Y3: 25MHz, mylib:CRYSTAL
- C10: value 1uF -> (none); device SparkFun:CAP0805 -> SparkFun:CAP_POLD
- C18: value 100nF -> 18p
- C2, C3: value 12pF -> 5p
- C21: value 10uF -> 18p
- C8, C9: value 1uF -> 100nF
- IC2: value KSZ8001L -> MIC4680; device mylib:KSZ8001L -> BillPorter:MIC4680
- R13: value 4.7k -> 10k
- R15: value 10k -> (none)
- R16: value 2.2k -> (none)
- R20: value 10k -> 47k
- R21: value (none) -> 330
- R6: value 6.65k -> 6.49k
- Y1: device crystal:CRYSTALTC26V -> mylib:CRYSTALXTAL003000-85SMX
Connections:
- net N$4 renamed HV
- removed net N$39: Q2.D, R21.1
- new net BTN1: IC1.P1[29]/MCOB2/PCAP1[1]/MAT0[1]
- new net ENET_RST: C17.1, IC1.P0[8]/I2STX_WS/MISO1/MAT2[2], IC3.RST#, R14.1
- new net LED1: IC1.P3[25]/MAT0[0]/PWM1[2], R21.2
- new net N$4: R27.1, USB.A
- new net N$43: D2.C, IC2.SW, L1.1
- new net N$44: IC1.RTCX2, R22.1
- new net N$7: PWR.A, R28.1
- new net USB_LED: IC1.P1[18]/USB_UP_LED/PWM1[1]/CAP1[0], R27.2
- net +3V3: now also IC3.VDDA_3.3, IC3.VDDIO, R13.2, R14.2, R28.2; no longer C17.1, C18.1, IC2.VDDIO, IC2.VDDRCV, IC6.VCC, LED1.A, R13.1, R14.1, R15.1, R16.1, U2.EN, U2.VCC
- net 5V: now also C10.+, L1.2, R15.1; no longer C24.+, IC5.VO
- net ENET_CRS: now also IC3.CRS_DV/CONFIG2; no longer IC2.RXDV/CRSDV/PCS_LPBK
- net ENET_LED_0: now also IC3.LED0/NWAYEN; no longer IC2.LED0/TEST
- net ENET_LED_1: now also IC3.LED1/SPEED; no longer IC2.LED1/SPD100/NOFEF
- net ENET_MDC: now also IC3.MDC; no longer IC2.MDC
- net ENET_MDIO: now also IC3.MDIO; no longer IC2.MDIO, R16.2
- net ENET_RD_N: now also IC3.RXM; no longer IC2.RX-
- net ENET_RD_P: now also IC3.RXP; no longer IC2.RX+
- net ENET_REF_CLK: now also IC3.REF_CLK/B-CAST_OFF; no longer IC2.TXC/REFCLK/CLOCK, IC6.Y
- net ENET_RXD0: now also IC3.RXD0/DUPLEX; no longer IC2.RXD0/RXD[0]/RX/PHYAD4
- net ENET_RXD1: now also IC3.RXD1/PHYAD2; no longer IC2.RXD1/RXD[1]/PHYAD3
- net ENET_RX_ER: now also IC3.RXER/ISO; no longer IC2.RXER/RX_ER/ISO
- net ENET_TD_N: now also IC3.TXM; no longer IC2.TX-
- net ENET_TD_P: now also IC3.TXP; no longer IC2.TX+
- net ENET_TXD0: now also IC3.TXD0; no longer IC2.TXD0/TXD[0]/TX
- net ENET_TXD1: now also IC3.TXD1; no longer IC2.TXD1/TXD[1]/SYNC
- net ENET_TX_EN: now also IC3.TXEN; no longer IC2.TXEN
- net GND: now also C10.-, C13.2, C25.2, C26.2, C8.2, C9.2, D2.A, IC2.SHDN, IC3.GND, IC3.NC, LED1.C, PWR.C, R16.1, USB.C; no longer C10.1, C24.-, C8.1, C9.1, IC2.GND, IC5.GND, IC6.GND, Q2.S, U2.GND
- net JP6_8: now also IC1.P0[10]/TXD2/SDA2/MAT3[0]; no longer IC1.P0[1]/TD1/RXD3/SCL1
- net JP6_9: now also IC1.P0[1]/TD1/RXD3/SCL1; no longer IC1.P0[10]/TXD2/SDA2/MAT3[0]
- net N$2: now also IC2.IN; no longer IC5.VI
- net N$23: now also Y1.1; no longer Y1.2
- net N$24: now also R22.2, Y1.2; no longer IC1.RTCX2, Y1.1
- net N$25: now also IC3.REXT, R6.2; no longer C10.2, C8.2, C9.2, IC2.VDDC, IC2.VDDPLL, IC2.VDDRX
- net N$28: now also C25.1, IC3.XI, Y3.2; no longer IC2.REXT, R6.2
- net N$30: now also C26.1, IC3.XO, Y3.1; no longer IC2.COL/RMII_SELECT, R13.2
- net N$32: now also C8.1, C9.1, IC3.VDD_1.2; no longer IC6.A, U2.OUT
- net N$37: now also IC3.CONFIG0, R13.1; no longer IC2.XI, R15.2
- net N$38: now also LED1.A, R21.1; no longer LED1.C, R21.2
- net N$42: now also IC2.FB, R15.2, R16.2; no longer IC1.P0[28]/SCL0/USB_SCL, Q2.G
- net RESET: now also C13.1
- net RSTOUT: now also IC1.P0[26]/AD0[3]/AOUT/RXD3; no longer C21.1, IC1.RSTOUT, IC2.RST#, R14.2
- net SWDCLK: now also IC1.TCK/SWDCLK
- net USB_D_N: now also C18.1
- net USB_D_P: now also C21.1
Other:
- note removed: "JP6-H: P0[0], P0[1], p0[10], P0[11]"
- moved on the sheet: BAT, C11, C17, C18, C2, C21, C23, C3, C8, C9, D1, J2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
